Commit message: needs some fixes damn

File: body.urdf (robot description, URDF)
Before this commit: robot robot, 4 links, 4 joints
Links:
- link Link0: geometry collision box size=[0.66399715] [0.49598595] [0.45054413]; visual box size=[0.66399715] [0.49598595] [0.45054413]
- link Link1: geometry collision box size=[0.39526619] [0.73433325] [0.88636962]; visual box size=[0.39526619] [0.73433325] [0.88636962]
- link Link2: geometry collision box size=[0.51721051] [0.21750592] [0.71008957]; visual box size=[0.51721051] [0.21750592] [0.71008957]
- link Link3: geometry collision box size=[0.52301243] [0.07801196] [0.66787524]; visual box size=[0.52301243] [0.07801196] [0.66787524]
Joints:
- joint Link0_Link1: axis 0.5024495757520382 0.923611205544766 0.19738952944707788 -> 0.22347911742616855 0.8167538291937597 0.6314123084276544; origin xyz=-0.5 0.0 0.0 rpy=0 0 0 -> xyz=0.0 -0.5 0.0 rpy=0 0 0
- joint Link1_Link2: axis 0.8363760901963991 0.728339944746367 0.8131809140555144 -> 0.07809105412602924 0.7619084169461309 0.006375869894509334; origin xyz=0 0 0 rpy=0 0 0 -> xyz=[0.39526619] 0 0 rpy=0 0 0
- joint Link2_Link3: axis 0.8939630541492931 0.04060828910877112 0.4269047765328381 -> 0.3170459054059972 0.12276605108136007 0.668497062529974; origin xyz=[0.83770248] 0 0 rpy=0 0 0 -> xyz=0 0 0 rpy=0 0 0
- joint Link3_Link4: axis 0.8574403047510781 0.5712487102127837 0.8275342515053522 -> 0.22387119126376376 0.09686903050885931 0.2994333939020569; origin xyz=0.5 0.0 0 rpy=0 0 0 -> xyz=0 0 0 rpy=0 0 0

Commit message: needs some more fixes

File: body.urdf (robot description, URDF)
Before this commit: robot robot, 4 links, 4 joints
Links:
- link Link0: geometry collision box size=[0.81772578] [0.5962216] [0.70052119]; visual box size=[0.81772578] [0.5962216] [0.70052119]
- link Link1: geometry collision box size=[0.13974824] [0.79597931] [0.13731358]; visual box size=[0.13974824] [0.79597931] [0.13731358]
- link Link2: geometry collision box size=[0.87873347] [0.23695095] [0.57207506]; visual box size=[0.87873347] [0.23695095] [0.57207506]
- link Link3: geometry collision box size=[0.16063814] [0.4046017] [0.24255236]; visual box size=[0.16063814] [0.4046017] [0.24255236]
Joints:
- joint Link0_Link1: axis 0.22347911742616855 0.8167538291937597 0.6314123084276544 -> 0.8987975770125884 0.39692006319468487 0.26458382636385425; origin xyz=0.0 -0.5 0.0 rpy=0 0 0 -> xyz=0.5 0.0 0.0 rpy=0 0 0
- joint Link1_Link2: axis 0.07809105412602924 0.7619084169461309 0.006375869894509334 -> 0.051183218455036816 0.47273695962286444 0.8110987913059918; origin xyz=[0.39526619] 0 0 rpy=0 0 0 -> xyz=[0.13974824] 0 0 rpy=0 0 0
- joint Link2_Link3: axis 0.3170459054059972 0.12276605108136007 0.668497062529974 -> 0.3191504120026186 0.899127490612413 0.059040578302476; origin xyz=0 0 0 rpy=0 0 0 -> xyz=[0.87873347] 0 0 rpy=0 0 0
- joint Link3_Link4: axis 0.22387119126376376 0.09686903050885931 0.2994333939020569 -> 0.7768083340038537 0.6827096778567685 0.03508722808116116; origin xyz=0 0 0 rpy=0 0 0 -> xyz=[0.16063814] 0 0 rpy=0 0 0

Commit message: bug fixes

File: body.urdf (robot description, URDF)
Before this commit: robot robot, 4 links, 4 joints
Links:
- link Link0: geometry collision box size=[0.19748919] [0.49658598] [0.88551836]; visual box size=[0.19748919] [0.49658598] [0.88551836]
- link Link1: geometry collision box size=[0.27385373] [0.22800775] [0.17521889]; visual box size=[0.27385373] [0.22800775] [0.17521889]
- link Link2: geometry collision box size=[0.70514692] [0.06978607] [0.6983955]; visual box size=[0.70514692] [0.06978607] [0.6983955]
- link Link3: geometry collision box size=[0.24530755] [0.84445473] [0.07975814]; visual box size=[0.24530755] [0.84445473] [0.07975814]
Joints:
- removed joint Link3_Link4
- joint Link0_Link1: axis 0.8987975770125884 0.39692006319468487 0.26458382636385425 -> 0.30624119326696986 0.936143883912821 0.8945651516116725; origin xyz=0.5 0.0 0.0 rpy=0 0 0 -> xyz=-0.5 0.0 0.0 rpy=0 0 0
- joint Link1_Link2: axis 0.051183218455036816 0.47273695962286444 0.8110987913059918 -> 0.46842775508105994 0.3015973188343707 0.8049836270189423; origin xyz=[0.13974824] 0 0 rpy=0 0 0 -> xyz=0 0 0 rpy=0 0 0
- joint Link2_Link3: axis 0.3191504120026186 0.899127490612413 0.059040578302476 -> 0.885240200511381 0.9981482078697654 0.7155771201730136; origin xyz=[0.87873347] 0 0 rpy=0 0 0 -> xyz=[0.70514692] 0 0 rpy=0 0 0

Commit message: Improved code

File: body.urdf (robot description, URDF)
Before this commit: robot robot, 4 links, 3 joints
Links:
- link Link0: geometry collision box size=[0.65339018] [0.19630989] [0.08028267]; visual box size=[0.65339018] [0.19630989] [0.08028267]
- link Link1: geometry collision box size=[0.04669655] [0.07391839] [0.80237337]; visual box size=[0.04669655] [0.07391839] [0.80237337]
- link Link2: geometry collision box size=[0.50483371] [0.19567718] [0.96953198]; visual box size=[0.50483371] [0.19567718] [0.96953198]
- link Link3: geometry collision box size=[0.1375247] [0.6865479] [0.36437506]; visual box size=[0.1375247] [0.6865479] [0.36437506]
Joints:
- joint Link0_Link1: axis 0.30624119326696986 0.936143883912821 0.8945651516116725 -> 0.13765932742999853 0.1463372056547706 0.7018219426332646; origin xyz=-0.5 0.0 0.0 rpy=0 0 0 -> xyz=0.0 0.5 0.0 rpy=0 0 0
- joint Link1_Link2: axis 0.46842775508105994 0.3015973188343707 0.8049836270189423 -> 0.382223400290278 0.11264426230402369 0.16795269470884355; origin xyz=0 0 0 rpy=0 0 0 -> xyz=[0.04669655] 0 0 rpy=0 0 0
- joint Link2_Link3: axis 0.885240200511381 0.9981482078697654 0.7155771201730136 -> 0.027270159003241812 0.7561537804209734 0.41319310892432826; origin xyz=[0.70514692] 0 0 rpy=0 0 0 -> xyz=[0.50483371] 0 0 rpy=0 0 0

Commit message: Revamped for assignment 8

File: body.urdf (robot description, URDF)
Before this commit: robot robot, 3 links, 2 joints
Links:
- removed link BackLeg
- removed link FrontLeg
- removed link Torso
- added link Link0, mass 1; collision box size=1.1363164372307994 0.5606922367272579 1.3497366916272404; visual box size=1.1363164372307994 0.5606922367272579 1.3497366916272404
- added link Link1, mass 1; collision box size=1.3834989152433521 1.2550925165150488 0.674862494213544; visual box size=1.3834989152433521 1.2550925165150488 0.674862494213544
- added link Link1Link10, mass 1; collision box size=0.5972688071731962 0.8798951463007578 0.9429447168270024; visual box size=0.5972688071731962 0.8798951463007578 0.9429447168270024
- added link Link1Link11, mass 1; collision box size=0.5972688071731962 0.8798951463007578 0.9429447168270024; visual box size=0.5972688071731962 0.8798951463007578 0.9429447168270024
- added link Link1Link20, mass 1; collision box size=0.6431232572741836 0.7453647939154007 0.8470810480738206; visual box size=0.6431232572741836 0.7453647939154007 0.8470810480738206
- added link Link1Link21, mass 1; collision box size=0.6431232572741836 0.7453647939154007 0.8470810480738206; visual box size=0.6431232572741836 0.7453647939154007 0.8470810480738206
Joints:
- removed joint Torso_BackLeg
- removed joint Torso_FrontLeg
- added joint Link0_Link1: type revolute, parent Link0, child Link1, origin xyz=0 0.28034611836362894 0.6748683458136202 rpy=0 0 0, axis 0 1 0, limit lower=-3.14159 upper=3.14159 effort=0.0 velocity=0.0
- added joint Link1Link10_Link1Link11: type revolute, parent Link1Link10, child Link1Link11, origin xyz=-0.5972688071731962 0.0 0.0 rpy=0 0 0, axis 0 1 0, limit lower=-3.14159 upper=3.14159 effort=0.0 velocity=0.0
- added joint Link1Link20_Link1Link21: type revolute, parent Link1Link20, child Link1Link21, origin xyz=0.0 0.0 0.8470810480738206 rpy=0 0 0, axis 0 1 0, limit lower=-3.14159 upper=3.14159 effort=0.0 velocity=0.0
- added joint Link1_Link1Link10: type revolute, parent Link1, child Link1Link10, origin xyz=-0.6917494576216761 0.6275462582575244 0.0 rpy=0 0 0, axis 0 1 0, limit lower=-3.14159 upper=3.14159 effort=0.0 velocity=0.0
- added joint Link1_Link1Link20: type revolute, parent Link1, child Link1Link20, origin xyz=0.0 0.6275462582575244 0.337431247106772 rpy=0 0 0, axis 0 1 0, limit lower=-3.14159 upper=3.14159 effort=0.0 velocity=0.0

Commit message: minor change

File: body.urdf (robot description, URDF)
Before this commit: robot robot, 6 links, 5 joints
Links:
- removed link Link1Link20
- removed link Link1Link21
- added link Link1Link00, mass 1; collision box size=0.9860955459757195 0.6631536192507164 0.968737357353437; visual box size=0.9860955459757195 0.6631536192507164 0.968737357353437
- added link Link1Link01, mass 1; collision box size=0.9860955459757195 0.6631536192507164 0.968737357353437; visual box size=0.9860955459757195 0.6631536192507164 0.968737357353437
- link Link0: geometry collision box size=1.273688055232157 1.065368889112507 1.0274652370754702; visual box size=1.273688055232157 1.065368889112507 1.0274652370754702
- link Link1: geometry collision box size=0.7270311513175912 0.731495813503969 1.4063017115685912; visual box size=0.7270311513175912 0.731495813503969 1.4063017115685912
- link Link1Link10: geometry collision box size=0.5461137996032636 0.731495813503969 0.937974863560076; visual box size=0.5461137996032636 0.731495813503969 0.937974863560076
- link Link1Link11: geometry collision box size=0.5461137996032636 0.8096595782409335 0.937974863560076; visual box size=0.5461137996032636 0.8096595782409335 0.937974863560076
Joints:
- removed joint Link1Link20_Link1Link21
- removed joint Link1_Link1Link20
- added joint Link1Link00_Link1Link01: type revolute, parent Link1Link00, child Link1Link01, origin xyz=0.9860955459757195 0.0 0.0 rpy=0 0 0, axis 0 1 0, limit lower=-3.14159 upper=3.14159 effort=0.0 velocity=0.0
- added joint Link1_Link1Link00: type revolute, parent Link1, child Link1Link00, origin xyz=0.3635155756587956 0.3657479067519845 0.0 rpy=0 0 0, axis 0 1 0, limit lower=-3.14159 upper=3.14159 effort=0.0 velocity=0.0
- joint Link0_Link1: origin xyz=0 0.28034611836362894 0.6748683458136202 rpy=0 0 0 -> xyz=0 0.5326844445562535 0.7031508557842956 rpy=0 0 0
- joint Link1Link10_Link1Link11: origin xyz=-0.5972688071731962 0.0 0.0 rpy=0 0 0 -> xyz=-0.5461137996032636 0.0 0.0 rpy=0 0 0
- joint Link1_Link1Link10: origin xyz=-0.6917494576216761 0.6275462582575244 0.0 rpy=0 0 0 -> xyz=-0.3635155756587956 0.3657479067519845 0.0 rpy=0 0 0
